File: DAQ-32-BNC-FR4.kicad_pcb (KiCad board)
At the start: 2 copper layers, 482.6 x 88.9 mm, 38 parts, among them J1 Conn_Coaxial, J10 Conn_Coaxial, J11 Conn_Coaxial, J12 Conn_Coaxial, J13 Conn_Coaxial, J14 Conn_Coaxial, J15 Conn_Coaxial, J16 Conn_Coaxial, J17 Conn_Coaxial, J18 Conn_Coaxial, J19 Conn_Coaxial, J2 Conn_Coaxial, J20 Conn_Coaxial, J21 Conn_Coaxial, J22 Conn_Coaxial, J23 Conn_Coaxial, J24 Conn_Coaxial, J25 Conn_Coaxial, J26 Conn_Coaxial, J27 Conn_Coaxial, J28 Conn_Coaxial, J29 Conn_Coaxial, J3 Conn_Coaxial, J30 Conn_Coaxial, J31 Conn_Coaxial, J32 Conn_Coaxial, J33 DB37, J34 DB37, J4 Conn_Coaxial, J5 Conn_Coaxial, J6 Conn_Coaxial, J7 Conn_Coaxial, J8 Conn_Coaxial, J9 Conn_Coaxial

Commit message: update
Parts:
- added Logo1: Logo_Open_Hardware_Small, 0local:Logo_2X, F.Cu at (152.4, 203.2)
